File: ae-bbc-pcb/ae-bbc-pcb.kicad_pcb (KiCad board)
At the start: 2 copper layers, 138.4 x 66.5 mm, 21 parts, among them J1 Conn_01x02_Pin, J10 Conn_01x02_Pin, J11 Conn_01x02_Pin, J12 Conn_01x02_Pin, J13 Conn_01x02_Pin, J14 Conn_01x02_Pin, J15 Conn_01x02_Pin, J16 Conn_01x02_Pin, J2 Conn_01x02_Pin, J3 Conn_01x02_Pin, J4 Conn_01x02_Pin, J5 Conn_01x02_Pin, J6 Conn_01x02_Pin, J7 Conn_01x02_Pin, J8 Conn_01x02_Pin, J9 Conn_01x02_Pin

Commit message: REV 0.1 to JLCPCB
Parts:
- J1: footprint Acea:AMASS_XT60PW-F_1x02_P7.20mm_Horizontal -> Acea:AMASS_XT60PW-M_1x02_P7.20mm_Horizontal
- J10, J11, J12, J13, J14, J15, J16, J2, J3, J4, J5, J6, J7, J8, J9: footprint Acea:AMASS_XT60PW-M_1x02_P7.20mm_Horizontal -> Connector_AMASS:AMASS_XT30PW-M_1x02_P2.50mm_Horizontal
- moved H1 11.7 mm to (153.7, 129.5)
- moved H3 11.7 mm to (153.7, 154.9)
- moved H2 10.5 mm to (255.3, 129.5)
- moved H4 10.5 mm to (255.3, 154.9)
- moved J2 7.52 mm to (259.8, 144.7)
- moved J11 7.36 mm to (221.4, 162.6)
- moved J15 7.36 mm to (262.1, 162.6)
- moved J3 7.36 mm to (140.2, 162.6)
- moved J13 7.36 mm to (241.8, 162.6)
- moved J5 7.36 mm to (160.5, 162.6)
- moved J7 7.36 mm to (180.8, 162.6)
- moved J9 7.36 mm to (201.1, 162.6)
- moved J1 7.20 mm to (143.3, 145.8)
- moved J10 7.08 mm to (206.2, 121.5)
- moved J12 7.08 mm to (226.5, 121.5)
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Other:
- board size 138.4 x 66.5 mm -> 138.9 x 66.5 mm
- board text added: "AE-BBC-D v0.1 (Big Beautiful Charger) (Distributor)"
- board text removed: "AE-BBC v0.1 (Big Beautiful Charger)"

Commit message: v0.2 waiting for feedback
Parts:
- removed G***: LOGO, Acea:ae_40mm
- added J17: Conn_01x02_Pin, Connector_JST:JST_XH_B2B-XH-A_1x02_P2.50mm_Vertical, F.Cu at (142.0, 129.0)
- added J18: Conn_01x02_Pin, Connector_JST:JST_XH_B2B-XH-A_1x02_P2.50mm_Vertical, F.Cu at (162.5, 129.0)
- added J19: Conn_01x02_Pin, Connector_JST:JST_XH_B2B-XH-A_1x02_P2.50mm_Vertical, F.Cu at (182.5, 129.0)
- added J20: Conn_01x02_Pin, Connector_JST:JST_XH_B2B-XH-A_1x02_P2.50mm_Vertical, F.Cu at (202.5, 129.0)
- added J21: Conn_01x02_Pin, Connector_JST:JST_XH_B2B-XH-A_1x02_P2.50mm_Vertical, F.Cu at (222.5, 129.0)
- added J22: Conn_01x02_Pin, Connector_JST:JST_XH_B2B-XH-A_1x02_P2.50mm_Vertical, F.Cu at (243.0, 129.0)
- added J23: Conn_01x02_Pin, Connector_JST:JST_XH_B2B-XH-A_1x02_P2.50mm_Vertical, F.Cu at (264.0, 129.0)
- added J24: Conn_01x02_Pin, Connector_JST:JST_XH_B2B-XH-A_1x02_P2.50mm_Vertical, F.Cu at (266.5, 155.0)
- added J25: Conn_01x02_Pin, Connector_JST:JST_XH_B2B-XH-A_1x02_P2.50mm_Vertical, F.Cu at (245.5, 155.0)
- added J26: Conn_01x02_Pin, Connector_JST:JST_XH_B2B-XH-A_1x02_P2.50mm_Vertical, F.Cu at (225.0, 155.0)
- added J27: Conn_01x02_Pin, Connector_JST:JST_XH_B2B-XH-A_1x02_P2.50mm_Vertical, F.Cu at (204.5, 155.0)
- added J28: Conn_01x02_Pin, Connector_JST:JST_XH_B2B-XH-A_1x02_P2.50mm_Vertical, F.Cu at (185.0, 155.0)
- added J29: Conn_01x02_Pin, Connector_JST:JST_XH_B2B-XH-A_1x02_P2.50mm_Vertical, F.Cu at (164.5, 155.0)
- added J30: Conn_01x02_Pin, Connector_JST:JST_XH_B2B-XH-A_1x02_P2.50mm_Vertical, F.Cu at (144.5, 155.0)
- J1: footprint Acea:AMASS_XT60PW-M_1x02_P7.20mm_Horizontal -> Acea:AMASS_XT60PW-F_1x02_P7.20mm_Horizontal
- moved J1 7.20 mm to (143.3, 138.6)
Other:
- board size 138.9 x 66.5 mm -> 138.4 x 66.3 mm
- board text added: "AE-BBC-D v0.2 (Big Beautiful Charger) (Distributor)"
- board text removed: "AE-BBC-D v0.1 (Big Beautiful Charger) (Distributor)"
