File: ae-bbc-pcb/ae-bbc-pcb.kicad_sch (KiCad schematic)
At the start: 20 parts, among them J1 Conn_01x02_Pin, J10 Conn_01x02_Pin, J11 Conn_01x02_Pin, J12 Conn_01x02_Pin, J13 Conn_01x02_Pin, J14 Conn_01x02_Pin, J15 Conn_01x02_Pin, J16 Conn_01x02_Pin, J2 Conn_01x02_Pin, J3 Conn_01x02_Pin, J4 Conn_01x02_Pin, J5 Conn_01x02_Pin, J6 Conn_01x02_Pin, J7 Conn_01x02_Pin, J8 Conn_01x02_Pin, J9 Conn_01x02_Pin

Commit message: REV 0.1 to JLCPCB
Parts:
- J1: footprint Acea:AMASS_XT60PW-F_1x02_P7.20mm_Horizontal -> Acea:AMASS_XT60PW-M_1x02_P7.20mm_Horizontal
- J10, J11, J12, J13, J14, J15, J16, J2, J3, J4, J5, J6, J7, J8, J9: footprint Acea:AMASS_XT60PW-M_1x02_P7.20mm_Horizontal -> Connector_AMASS:AMASS_XT30PW-M_1x02_P2.50mm_Horizontal; lcsc C98732 -> C431092
Changed lines of the file:
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@@
 			)
 		)
-		(property "Footprint" "Acea:AMASS_XT60PW-M_1x02_P7.20mm_Horizontal"
+		(property "Footprint" "Connector_AMASS:AMASS_XT30PW-M_1x02_P2.50mm_Horizontal"
 			(at 141.986 128.016 0)
 			(effects
@@
 			)
 		)
-		(property "lcsc" "C98732"
+		(property "lcsc" "C431092"
 			(at 141.986 128.016 0)
 			(effects
@@
 			)
 		)
-		(property "Footprint" "Acea:AMASS_XT60PW-M_1x02_P7.20mm_Horizontal"
+		(property "Footprint" "Connector_AMASS:AMASS_XT30PW-M_1x02_P2.50mm_Horizontal"
 			(at 166.624 114.046 0)
 			(effects
@@
 			)
 		)
-		(property "lcsc" "C98732"
+		(property "lcsc" "C431092"
 			(at 166.624 114.046 0)
 			(effects
@@
 			)
 		)
-		(property "Footprint" "Acea:AMASS_XT60PW-M_1x02_P7.20mm_Horizontal"
+		(property "Footprint" "Connector_AMASS:AMASS_XT30PW-M_1x02_P2.50mm_Horizontal"
 			(at 114.808 114.046 0)
 			(effects
@@
 			)
 		)
-		(property "lcsc" "C98732"
+		(property "lcsc" "C431092"
 			(at 114.808 114.046 0)
 			(effects
@@
 			)
 		)
-		(property "Footprint" "Acea:AMASS_XT60PW-M_1x02_P7.20mm_Horizontal"
+		(property "Footprint" "Connector_AMASS:AMASS_XT30PW-M_1x02_P2.50mm_Horizontal"
 			(at 114.808 107.442 0)
 			(effects
@@
 			)
 		)
-		(property "lcsc" "C98732"
+		(property "lcsc" "C431092"
 			(at 114.808 107.442 0)
 			(effects
@@
 			)
 		)
-		(property "Footprint" "Acea:AMASS_XT60PW-M_1x02_P7.20mm_Horizontal"
+		(property "Footprint" "Connector_AMASS:AMASS_XT30PW-M_1x02_P2.50mm_Horizontal"
 			(at 115.062 87.884 0)
 			(effects
@@
 			)
 		)
-		(property "lcsc" "C98732"
+		(property "lcsc" "C431092"
 			(at 115.062 87.884 0)
 			(effects
@@
 			)
 		)
-		(property "Footprint" "Acea:AMASS_XT60PW-M_1x02_P7.20mm_Horizontal"
+		(property "Footprint" "Connector_AMASS:AMASS_XT30PW-M_1x02_P2.50mm_Horizontal"
 			(at 166.624 107.442 0)
 			(effects
@@
 			)
 		)
-		(property "lcsc" "C98732"
+		(property "lcsc" "C431092"
 			(at 166.624 107.442 0)
 			(effects
@@
 			)
 		)
-		(property "Footprint" "Acea:AMASS_XT60PW-M_1x02_P7.20mm_Horizontal"
+		(property "Footprint" "Connector_AMASS:AMASS_XT30PW-M_1x02_P2.50mm_Horizontal"
 			(at 166.37 100.838 0)
 			(effects
@@
 			)
 		)
-		(property "lcsc" "C98732"
+		(property "lcsc" "C431092"
 			(at 166.37 100.838 0)
 			(effects
@@
 			)
 		)
-		(property "Footprint" "Acea:AMASS_XT60PW-M_1x02_P7.20mm_Horizontal"
+		(property "Footprint" "Connector_AMASS:AMASS_XT30PW-M_1x02_P2.50mm_Horizontal"
 			(at 114.808 120.396 0)
 			(effects
@@
 			)
 		)
-		(property "lcsc" "C98732"
+		(property "lcsc" "C431092"
 			(at 114.808 120.396 0)
 			(effects
@@
 			)
 		)
-		(property "Footprint" "Acea:AMASS_XT60PW-F_1x02_P7.20mm_Horizontal"
+		(property "Footprint" "Acea:AMASS_XT60PW-M_1x02_P7.20mm_Horizontal"
 			(at 141.986 67.818 0)
 			(effects
@@
 			)
 		)
-		(property "Footprint" "Acea:AMASS_XT60PW-M_1x02_P7.20mm_Horizontal"
+		(property "Footprint" "Connector_AMASS:AMASS_XT30PW-M_1x02_P2.50mm_Horizontal"
 			(at 166.37 87.884 0)
 			(effects
@@
 			)
 		)
-		(property "lcsc" "C98732"
+		(property "lcsc" "C431092"
 			(at 166.37 87.884 0)
 			(effects
@@
 			)
 		)
-		(property "Footprint" "Acea:AMASS_XT60PW-M_1x02_P7.20mm_Horizontal"
+		(property "Footprint" "Connector_AMASS:AMASS_XT30PW-M_1x02_P2.50mm_Horizontal"
 			(at 115.316 81.28 0)
 			(effects
@@
 			)
 		)
-		(property "lcsc" "C98732"
+		(property "lcsc" "C431092"
 			(at 115.316 81.28 0)
 			(effects
@@
 			)
 		)
-		(property "Footprint" "Acea:AMASS_XT60PW-M_1x02_P7.20mm_Horizontal"
+		(property "Footprint" "Connector_AMASS:AMASS_XT30PW-M_1x02_P2.50mm_Horizontal"
 			(at 115.062 100.838 0)
 			(effects
@@
 			)
 		)
-		(property "lcsc" "C98732"
+		(property "lcsc" "C431092"
 			(at 115.062 100.838 0)
 			(effects
@@
 			)
 		)
-		(property "Footprint" "Acea:AMASS_XT60PW-M_1x02_P7.20mm_Horizontal"
+		(property "Footprint" "Connector_AMASS:AMASS_XT30PW-M_1x02_P2.50mm_Horizontal"
 			(at 166.624 120.396 0)
 			(effects
@@
 			)
 		)
-		(property "lcsc" "C98732"
+		(property "lcsc" "C431092"
 			(at 166.624 120.396 0)
 			(effects
@@
 			)
 		)
-		(property "Footprint" "Acea:AMASS_XT60PW-M_1x02_P7.20mm_Horizontal"
+		(property "Footprint" "Connector_AMASS:AMASS_XT30PW-M_1x02_P2.50mm_Horizontal"
 			(at 166.116 81.28 0)
 			(effects
@@
 			)
 		)
-		(property "lcsc" "C98732"
+		(property "lcsc" "C431092"
 			(at 166.116 81.28 0)
 			(effects
@@
 			)
 		)
-		(property "Footprint" "Acea:AMASS_XT60PW-M_1x02_P7.20mm_Horizontal"
+		(property "Footprint" "Connector_AMASS:AMASS_XT30PW-M_1x02_P2.50mm_Horizontal"
 			(at 115.062 94.488 0)
 			(effects
@@
 			)
 		)
-		(property "lcsc" "C98732"
+		(property "lcsc" "C431092"
 			(at 115.062 94.488 0)
 			(effects
@@
 			)
 		)
-		(property "Footprint" "Acea:AMASS_XT60PW-M_1x02_P7.20mm_Horizontal"
+		(property "Footprint" "Connector_AMASS:AMASS_XT30PW-M_1x02_P2.50mm_Horizontal"
 			(at 166.37 94.488 0)
 			(effects
@@
 			)
 		)
-		(property "lcsc" "C98732"
+		(property "lcsc" "C431092"
 			(at 166.37 94.488 0)
 			(effects

Commit message: v0.2 waiting for feedback
Parts:
- added J17, J18, J19, J20, J21, J22, J23, J24, J25, J26, J27, J28, J29, J30: Conn_01x02_Pin, Connector_JST:JST_XH_B2B-XH-A_1x02_P2.50mm_Vertical, symbol Connector:Conn_01x02_Pin
- J1: footprint Acea:AMASS_XT60PW-M_1x02_P7.20mm_Horizontal -> Acea:AMASS_XT60PW-F_1x02_P7.20mm_Horizontal
Connections:
- net at J1.1 (Pin_1), J10.1 (Pin_1), J11.1 (Pin_1)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: now also J17.2 (Pin_2), J18.2 (Pin_2), J19.2 (Pin_2), J20.2 (Pin_2), J21.2 (Pin_2), J22.2 (Pin_2), J23.2 (Pin_2), J24.2 (Pin_2), J25.2 (Pin_2), J26.2 (Pin_2), J27.2 (Pin_2), J28.2 (Pin_2), J29.2 (Pin_2), J30.2 (Pin_2)
- net at J1.2 (Pin_2), J10.2 (Pin_2), J11.2 (Pin_2)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: now also J17.1 (Pin_1), J18.1 (Pin_1), J19.1 (Pin_1), J20.1 (Pin_1), J21.1 (Pin_1), J22.1 (Pin_1), J23.1 (Pin_1), J24.1 (Pin_1), J25.1 (Pin_1), J26.1 (Pin_1), J27.1 (Pin_1), J28.1 (Pin_1), J29.1 (Pin_1), J30.1 (Pin_1)
